File: pcb/keybed.kicad_sch (KiCad schematic)
At the start: 27 parts, among them J1 I/0, J2 Programmer, J3 AT, J5 Keyboard, J6 Midi, U1 ATMega328p, U2 74HC164, U3 74HC165, U4 74HC165, Y1 16MHz

Commit message: Added schematic and files to build case
Other:
- title: (none) -> Matrix Scanner
Changed lines of the file:
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@@
 (kicad_sch (version 20211123) (generator eeschema)
   (paper "A4")
+  (title_block
+    (title "Matrix Scanner")
+  )
   (junction (at 167.64 69.85) (diameter 0) (color 0 0 0 0)
   )
